Commit message: corrected orientation of mount to grippers when mounted in higher level urdf.

File: ezgripper_description/urdf/SAKE_double_mount.urdf.xacro (robot description, xacro)
@@ -4,5 +4,5 @@
 		<!-- links -->
 		<joint name="${prefix}_ezgripper_mount2base" type="fixed">
-				<origin rpy="0 0 0" xyz="0.0 0.0 0.0"/>
+				<xacro:insert_block name="origin"/>
 				<parent link="${parent_link}"/>
 				<child link="${prefix}_ezgripper_to_mount"/>
@@ -12,5 +12,5 @@
 		<link name="${prefix}_ezgripper_to_mount">
 			<visual>
-				<xacro:insert_block name="origin"/>
+				<origin rpy="0 0 0" xyz="0.0 0.0 0.0"/>
 				<geometry>
 					<mesh filename="file://$(find ezgripper_description)/meshes/visual/SAKE_Double_Mount.stl"/>
@@ -19,5 +19,5 @@
 			</visual>
 			<collision>
-				<xacro:insert_block name="origin"/>
+				<origin rpy="0 0 0" xyz="0.0 0.0 0.0"/>
 				<geometry>
 					<mesh filename="file://$(find ezgripper_description)/meshes/collision/SAKE_Double_Mount.stl"/>

File: ezgripper_description/urdf/SAKE_single_mount.urdf.xacro (robot description, xacro)
@@ -4,5 +4,5 @@
 		<!-- links -->
 		<joint name="${prefix}_ezgripper_mount2base" type="fixed">
-				<origin rpy="0 0 0" xyz="0.0 0.0 0.0"/>
+				<xacro:insert_block name="origin"/>
 				<parent link="${parent_link}"/>
 				<child link="${prefix}_ezgripper_to_mount"/>
@@ -12,5 +12,5 @@
 		<link name="${prefix}_ezgripper_to_mount">
 			<visual>
-				<xacro:insert_block name="origin"/>
+				<origin rpy="0 0 0" xyz="0.0 0.0 0.0"/>
 				<geometry>
 					<mesh filename="file://$(find ezgripper_description)/meshes/visual/SAKE_Single_Mount.stl"/>
@@ -19,5 +19,5 @@
 			</visual>
 			<collision>
-				<xacro:insert_block name="origin"/>
+				<origin rpy="0 0 0" xyz="0.0 0.0 0.0"/>
 				<geometry>
 					<mesh filename="file://$(find ezgripper_description)/meshes/collision/SAKE_Single_Mount.stl"/>

File: ezgripper_description/urdf/SAKE_triple_mount.urdf.xacro (robot description, xacro)
@@ -4,5 +4,5 @@
 		<!-- links -->
 		<joint name="${prefix}_ezgripper_mount2base" type="fixed">
-				<origin rpy="0 0 0" xyz="0.0 0.0 0.0"/>
+				<xacro:insert_block name="origin"/>
 				<parent link="${parent_link}"/>
 				<child link="${prefix}_ezgripper_to_mount"/>
@@ -12,5 +12,5 @@
 		<link name="${prefix}_ezgripper_to_mount">
 			<visual>
-				<xacro:insert_block name="origin"/>
+				<origin rpy="0 0 0" xyz="0.0 0.0 0.0"/>
 				<geometry>
 					<mesh filename="file://$(find ezgripper_description)/meshes/visual/SAKE_Triple_Mount.stl"/>
@@ -19,5 +19,5 @@
 			</visual>
 			<collision>
-				<xacro:insert_block name="origin"/>
+				<origin rpy="0 0 0" xyz="0.0 0.0 0.0"/>
 				<geometry>
 					<mesh filename="file://$(find ezgripper_description)/meshes/collision/SAKE_Triple_Mount.stl"/>
